File: latest/iium_sumo.kicad_pcb (KiCad board)
At the start: 2 copper layers, 100 x 60 mm, 59 parts, among them J1 I2C_VL53_1, J10 Cytron MD, J11 Cytron Start Module, J12 Conn_01x04, J13 Conn_01x04, J14 Conn_01x04, J15 EXTRA1, J16 Conn_01x02_Pin, J17 Conn_01x02_Pin, J18 UART1, J19 UART2, J2 I2C_VL53_2, J3 I2C_VL53_3, J4 I2C_VL53_4, J5 I2C_VL53_5, J6 IR_1, J7 IR_2, J8 IR_3, J9 IR_4, SW1 SW_SPST, SW2 SW_SPST, SW3 SW_SPDT, U1 TPS54360DDA, U4 Black Pill v2, U5 LM3940

Commit message: relayout button
Parts:
- added REF**: MountingHole_3.5mm, MountingHole:MountingHole_3.5mm, F.Cu at (104.5, 112.0)
- moved C17 42.9 mm to (106.5, 73.0), turned to 90 degrees
- moved SW2 37.4 mm to (102.8, 75.2), turned to 90 degrees
- moved R4 26.9 mm to (106.5, 79.1)
- moved R3 22.9 mm to (106.5, 91.3), turned to -90 degrees
- moved SW1 12.9 mm to (102.8, 95.2), turned to -90 degrees
- moved C16 7.02 mm to (106.5, 97.4), turned to -90 degrees
- moved REF** 2.73 mm to (104.5, 63.0)
- moved REF** 2.73 mm to (193.5, 63.0)
- moved REF** 2.73 mm to (193.5, 112.0)
- moved C1 1.51 mm to (189.5, 85.5)
- moved C11 1.51 mm to (185.8, 72.6)
- moved C12 1.51 mm to (177.9, 82.9)
- moved C14 1.51 mm to (178.3, 95.7)
- moved C3 1.51 mm to (189.5, 90.5)
- moved C5 1.51 mm to (177.9, 80.3)
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Routing:
- net +3V3: track 260.7 -> 206.0 mm, vias 0 -> 3
- net /PB13: track 19.7 -> 28.4 mm
- net /PB12: track 20.9 -> 13.3 mm
- net GND: vias 45 -> 74
